File: Kicad - Projects/Inv_Spot_Pot/Inv_Spot_Pot.kicad_sch (KiCad schematic)
At the start: 68 parts, among them J1 Screw_Terminal_01x03, J2 PWM, J3 Display_Power, J4 Current_Sense, J5 PWM, Q1 40T120, Q2 40T120, Q3 40T120, Q4 40T120, T1 Transformer_1P_2S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

Commit message: Melhoras na Ponte Completa
Placa de ponte completa quase feita, falta rotear os PWMs e adicionar o cabo que leva T- ao transformador

Removido arquivo .history devido a incomodar na hora de uppar os arquivos
Parts:
- added HS3: Heatsink, Custom_Footprints:Heatsink_17x15mm, symbol Mechanical:Heatsink
- HS2: footprint Heatsink:Heatsink_35x15mm -> Custom_Footprints:Heatsink_17x15mm
Connections:
- net Earth: now also T2.1, T2.3; no longer T2.2, T2.4
- net ~{PWM1}: now also T2.2; no longer T2.3
- net ~{PWM}: now also T2.4; no longer T2.1
Other:
- moved on the sheet: HS1, HS2, J2

Commit message: Ajustes Semi-Finais
Adicionados circuitos de gate e capacitores de polipropileno, falta apenas o footprint final do transformador e os capacitores de segurança em Y na fonte auxiliar e saída da linha AC
Connections:
- net Earth: now also T2.2; no longer T2.1
- net PWM: now also T2.7; no longer T2.6
- net PWM1: now also T2.6; no longer T2.8
- net T+: now also T2.5; no longer T2.7
- net T-: now also T2.8; no longer T2.5
- net ~{PWM1}: now also T2.4; no longer T2.2
- net ~{PWM}: now also T2.1; no longer T2.4
Changed lines of the file:
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@@
 	)
 	(junction
-		(at 260.35 50.8)
-		(diameter 0)
-		(color 0 0 0 0)
-	)
-	(junction
 		(at 64.77 101.6)
 		(diameter 0)
@@
 	)
 	(junction
+		(at 260.35 50.8)
+		(diameter 0)
+		(color 0 0 0 0)
+	)
+	(junction
 		(at 111.76 118.11)
 		(diameter 0)
@@
 	(wire
 		(pts
-			(xy 250.19 48.26) (xy 248.92 48.26)
-		)
-		(stroke
-			(width 0)
-			(type default)
-		)
-	)
-	(wire
-		(pts
 			(xy 106.68 44.45) (xy 90.17 44.45)
 		)
@@
 	(wire
 		(pts
+			(xy 248.92 38.1) (xy 250.19 38.1)
+		)
+		(stroke
+			(width 0)
+			(type default)
+		)
+	)
+	(wire
+		(pts
 			(xy 143.51 166.37) (xy 143.51 167.64)
 		)
@@
 	(wire
 		(pts
-			(xy 248.92 38.1) (xy 260.35 38.1)
-		)
-		(stroke
-			(width 0)
-			(type default)
-		)
-	)
-	(wire
-		(pts
 			(xy 237.49 152.4) (xy 237.49 147.32)
 		)
@@
 	(wire
 		(pts
+			(xy 260.35 48.26) (xy 260.35 50.8)
+		)
+		(stroke
+			(width 0)
+			(type default)
+		)
+	)
+	(wire
+		(pts
 			(xy 152.4 114.3) (xy 152.4 118.11)
 		)
@@
 	(wire
 		(pts
+			(xy 248.92 48.26) (xy 260.35 48.26)
+		)
+		(stroke
+			(width 0)
+			(type default)
+		)
+	)
+	(wire
+		(pts
 			(xy 215.9 142.24) (xy 215.9 147.32)
 		)
@@
 	(wire
 		(pts
-			(xy 260.35 38.1) (xy 260.35 50.8)
-		)
-		(stroke
-			(width 0)
-			(type default)
-		)
-	)
-	(wire
-		(pts
 			(xy 191.77 96.52) (xy 191.77 93.98)
 		)
@@
 	(global_label "~{PWM1}"
 		(shape input)
-		(at 250.19 48.26 0)
+		(at 250.19 38.1 0)
 		(fields_autoplaced yes)
 		(effects
@@
 		)
 		(property "Intersheetrefs" "${INTERSHEET_REFS}"
-			(at 258.5575 48.26 0)
+			(at 258.5575 38.1 0)
 			(hide yes)
 			(show_name no)

Commit message: Final - Placa Ponte Completa
Ajustadas todas as rotas da placa de potência por ponte completa, falta apenas adicionar test-points
Parts:
- added CY1, CY2, CY3: C, Capacitor_THT:C_Disc_D10.5mm_W5.0mm_P10.00mm, symbol Device:C
Connections:
- net Earth: now also CY3.1
- net GND: now also CY3.2
- net T+: now also TR1.1; no longer T1.2 (AB)
- net T-: now also T1.1 (AA); no longer TR1.1
- net at Cx2.1, D1.2, FL1.2: now also CY1.1
- net at Cx2.2, D1.3, FL1.4: now also CY2.2
- net at TR1.2: now also T1.2 (AB); no longer T1.1 (AA)
- new net Earth_Protective: CY1.2, CY2.1
Other:
- moved on the sheet: J4, TR1

Commit message: Adicionados Testpoints
Adicionados testpoints:
 - Gate de cada IGBT (+ emissor)
 - Tensão do barramento
 - Barramento da fonte auxiliar

Trocado footprint do sensor de corrente para pinheader
Parts:
- J4: footprint Connector_JST:JST_ZH_B2B-ZR_1x02_P1.50mm_Vertical -> Connector_PinHeader_2.00mm:PinHeader_1x02_P2.00mm_Vertical
Changed lines of the file:
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@@
 			)
 		)
-		(property "Footprint" "Connector_JST:JST_ZH_B2B-ZR_1x02_P1.50mm_Vertical"
+		(property "Footprint" "Connector_PinHeader_2.00mm:PinHeader_1x02_P2.00mm_Vertical"
 			(at 196.85 111.76 0)
 			(hide yes)

Commit message: Finalizada Placa de Potência
Capacitor de desacoplamento de 15V da fonte auxiliar movido para estar mais próximo da saída

Footprint do transformador corrigida

PWM da camada de cima afastado do dissipador de Q2

Maior afastamento entre planos GND/Earth e trilhas na fonte auxiliar

Modificado símbolo do transformador de saída no esquemático para melhor refletir a saída
Parts:
- removed T1: Transformer_1P_2S, Transformer_THT:Transformer_Toroid_THT_7032, symbol Device:Transformer_1P_2S
- added T1: Transformer_1P_1S, Transformer_THT:Transformer_Toroid_THT_7032, symbol Device:Transformer_1P_1S
Connections:
- net T-: now also T1.1 (AA)
- net at TR1.2: now also T1.2 (AB)
Changed lines of the file:
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@@
 	(wire
 		(pts
-			(xy 233.68 83.82) (xy 233.68 88.9)
-		)
-		(stroke
-			(width 0)
-			(type default)
-		)
-	)
-	(wire
-		(pts
 			(xy 92.71 33.02) (xy 92.71 34.29)
 		)
@@
 	(wire
 		(pts
-			(xy 232.41 83.82) (xy 233.68 83.82)
-		)
-		(stroke
-			(width 0)
-			(type default)
-		)
-	)
-	(wire
-		(pts
 			(xy 57.15 115.57) (xy 62.23 115.57)
 		)
@@
 	(wire
 		(pts
-			(xy 233.68 88.9) (xy 232.41 88.9)
-		)
-		(stroke
-			(width 0)
-			(type default)
-		)
-	)
-	(wire
-		(pts
 			(xy 72.39 101.6) (xy 64.77 101.6)
 		)
@@
 	)
 	(symbol
+		(lib_id "Device:Transformer_1P_1S")
+		(at 222.25 86.36 0)
+		(unit 1)
+		(body_style 1)
+		(exclude_from_sim no)
+		(in_bom yes)
+		(on_board yes)
+		(in_pos_files yes)
+		(dnp no)
+		(fields_autoplaced yes)
+		(property "Reference" "T1"
+			(at 222.2627 76.2 0)
+			(show_name no)
+			(do_not_autoplace no)
+			(effects
+				(font
+					(size 1.27 1.27)
+				)
+			)
+		)
+		(property "Value" "Transformer_1P_1S"
+			(at 222.2627 78.74 0)
+			(show_name no)
+			(do_not_autoplace no)
+			(effects
+				(font
+					(size 1.27 1.27)
+				)
+			)
+		)
+		(property "Footprint" "Transformer_THT:Transformer_Toroid_THT_7032"
+			(at 222.25 86.36 0)
+			(hide yes)
+			(show_name no)
+			(do_not_autoplace no)
+			(effects
+				(font
+					(size 1.27 1.27)
+				)
+			)
+		)
+		(property "Datasheet" ""
+			(at 222.25 86.36 0)
+			(hide yes)
+			(show_name no)
+			(do_not_autoplace no)
+			(effects
+				(font
+					(size 1.27 1.27)
+				)
+			)
+		)
+		(property "Description" "Transformer, single primary, single secondary"
+			(at 222.25 86.36 0)
+			(hide yes)
+			(show_name no)
+			(do_not_autoplace no)
+			(effects
+				(font
+					(size 1.27 1.27)
+				)
+			)
+		)
+		(pin "1"
+		)
+		(pin "4"
+		)
+		(pin "2"
+		)
+		(pin "3"
+		)
+		(instances
+			(project "Inv_Spot_Pot"
+				(path "/e27abe51-96c0-4fdf-ba00-b5a281cd0e9c"
+					(reference "T1")
+					(unit 1)
+				)
+			)
+		)
+	)
+	(symbol
 		(lib_id "power:Earth")
 		(at 97.79 36.83 0)
@@
 					(unit 1)
 				)
-			)
-		)
-	)
-	(symbol
-		(lib_id "Device:Transformer_1P_2S")
-		(at 222.25 86.36 0)
-		(unit 1)
-		(body_style 1)
-		(exclude_from_sim no)
-		(in_bom yes)
-		(on_board yes)
-		(in_pos_files yes)
-		(dnp no)
-		(fields_autoplaced yes)
-		(property "Reference" "T1"
-			(at 222.25 71.12 0)
-			(show_name no)
-			(do_not_autoplace no)
-			(effects
-				(font
-					(size 1.27 1.27)
-				)
-			)
-		)
-		(property "Value" "Transformer_1P_2S"
-			(at 222.25 73.66 0)
-			(show_name no)
-			(do_not_autoplace no)
-			(effects
-				(font
-					(size 1.27 1.27)
-				)
-			)
-		)
-		(property "Footprint" "Transformer_THT:Transformer_Toroid_THT_7032"
-			(at 222.25 86.36 0)
-			(hide yes)
-			(show_name no)
-			(do_not_autoplace no)
-			(effects
-				(font
-					(size 1.27 1.27)
-				)
-			)
-		)
-		(property "Datasheet" ""
-			(at 222.25 86.36 0)
-			(hide yes)
-			(show_name no)
-			(do_not_autoplace no)
-			(effects
-				(font
-					(size 1.27 1.27)
-				)
-			)
-		)
-		(property "Description" "Transformer, single primary, dual secondary"
-			(at 222.25 86.36 0)
-			(hide yes)
-			(show_name no)
-			(do_not_autoplace no)
-			(effects
-				(font
-					(size 1.27 1.27)
-				)
-			)
-		)
-		(pin "3"
-		)
-		(pin "6"
-		)
-		(pin "5"
-		)
-		(pin "4"
-		)
-		(pin "1"
-		)
-		(pin "2"
-		)
-		(instances
-			(project "Inv_Spot_Pot"
-				(path "/e27abe51-96c0-4fdf-ba00-b5a281cd0e9c"
-					(reference "T1")
-					(unit 1)
-				)

Commit message: Primeiro Layout - Display
Feito o layout preliminar da placa de display, conferir com o Anderson

Corrigido problema com o layout do transformador (erro no símbolo utilizado levou a inversão dos IGBTs superiores)
Connections:
- net PWM: now also T2.8; no longer T2.7
- net PWM1: now also T2.5; no longer T2.6
- net T+: now also T2.6; no longer T2.5
- net T-: now also T2.7; no longer T2.8

Commit message: Ajustes Finais
Ajustes em larguras de trilha da camada top

Ajuste do footprint dos capacitores de polipropileno dos IGBTs

Ajuste dos planos de referência
Parts:
- C15, C16, C17, C18: footprint Capacitor_THT:C_Rect_L7.2mm_W3.0mm_P5.00mm_FKS2_FKP2_MKS2_MKP2 -> Capacitor_THT:C_Rect_L11.0mm_W5.3mm_P10.00mm_MKT
Changed lines of the file:
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@@
 			)
 		)
-		(property "Footprint" "Capacitor_THT:C_Rect_L7.2mm_W3.0mm_P5.00mm_FKS2_FKP2_MKS2_MKP2"
+		(property "Footprint" "Capacitor_THT:C_Rect_L11.0mm_W5.3mm_P10.00mm_MKT"
 			(at 175.5648 45.72 0)
 			(hide yes)
@@
 			)
 		)
-		(property "Footprint" "Capacitor_THT:C_Rect_L7.2mm_W3.0mm_P5.00mm_FKS2_FKP2_MKS2_MKP2"
+		(property "Footprint" "Capacitor_THT:C_Rect_L11.0mm_W5.3mm_P10.00mm_MKT"
 			(at 157.1752 60.96 0)
 			(hide yes)
@@
 			)
 		)
-		(property "Footprint" "Capacitor_THT:C_Rect_L7.2mm_W3.0mm_P5.00mm_FKS2_FKP2_MKS2_MKP2"
+		(property "Footprint" "Capacitor_THT:C_Rect_L11.0mm_W5.3mm_P10.00mm_MKT"
 			(at 175.5648 62.23 0)
 			(hide yes)
@@
 			)
 		)
-		(property "Footprint" "Capacitor_THT:C_Rect_L7.2mm_W3.0mm_P5.00mm_FKS2_FKP2_MKS2_MKP2"
+		(property "Footprint" "Capacitor_THT:C_Rect_L11.0mm_W5.3mm_P10.00mm_MKT"
 			(at 157.1752 45.72 0)
 			(hide yes)
