File: Kicad - Projects/Inv_Spot_Pot/Inv_Spot_Pot - A.kicad_pcb (KiCad board)
At the start: 2 copper layers, 202.6 x 144.5 mm, 91 parts, among them J2 PWM, J3 Display_Power, J4 24V, K1 Y14x-1C-xxDS, Q1 40T120, Q2 40T120, Q3 40T120, Q4 40T120, T1 Transformer_1P_2S, U2 LTV-817S

Commit message: Atualização de Footprint
Atualizados footrpints do capacitor da fonte auxiliar e do transformador toroidal
Parts:
- added CY4: C, Capacitor_THT:C_Disc_D7.0mm_W2.5mm_P5.00mm, F.Cu at (260.4, 57.2)
- added CY5: C, Capacitor_THT:C_Disc_D7.0mm_W2.5mm_P5.00mm, F.Cu at (260.4, 61.3)
- added D22: DF06S, Diode_SMD:Diode_Bridge_OnSemi_SDIP-4L, F.Cu at (252.6, 60.1)
- added R24: 47, Resistor_SMD:R_2512_6332Metric, F.Cu at (242.3, 32.9)
- added R25: 47, Resistor_SMD:R_2512_6332Metric, F.Cu at (242.3, 37.8)
- added R26: 47, Resistor_SMD:R_2512_6332Metric, F.Cu at (242.3, 42.7)
- added R27: 47, Resistor_SMD:R_2512_6332Metric, F.Cu at (242.3, 47.6)
- added R28: 47, Resistor_SMD:R_2512_6332Metric, F.Cu at (242.3, 52.5)
- added R29: 47, Resistor_SMD:R_2512_6332Metric, F.Cu at (242.3, 57.4)
- added R30: 47, Resistor_SMD:R_2512_6332Metric, F.Cu at (242.3, 62.4)
- added R31: 47, Resistor_SMD:R_2512_6332Metric, F.Cu at (242.3, 67.3)
- added U3: ~, Custom_Transformer:EEL25V 6T+6T, F.Cu at (262.9, 88.1)
- C1, C2, C3, C4: value 220u -> 680u
- C10: value 47u -> 100u; footprint Capacitor_THT:CP_Radial_D8.0mm_P3.50mm -> Capacitor_THT:CP_Radial_D18.0mm_P7.50mm
- C13: value 47p -> 4.7n
- C15, C16, C17, C18: value 100n -> 4.7n; footprint Capacitor_THT:C_Rect_L11.0mm_W5.3mm_P10.00mm_MKT -> Capacitor_THT:C_Disc_D7.0mm_W2.5mm_P5.00mm
- C19, C20, C21, C22: value 100n -> 10n
- D21: footprint LED_THT:LED_D1.8mm_W3.3mm_H2.4mm -> LED_THT:LED_D5.0mm_Clear
- D4: footprint Diode_SMD:D_SOD-128 -> Diode_SMD:D_SMB
- F2, J4: footprint Connector_PinHeader_2.54mm:PinHeader_1x02_P2.54mm_Vertical -> Connector_JST:JST_XH_B2B-XH-A_1x02_P2.50mm_Vertical
- Q1, Q2, Q3, Q4: value 40T120 -> 60N60
Connections:
- C15 pad 1: 310V -> Net-(C15-Pad1)
- C16 pad 1: T- -> Net-(C16-Pad1)
- C17 pad 1: 310V -> Net-(C17-Pad1)
- C18 pad 1: T+ -> Net-(C18-Pad1)
- C20 pad 1: T- -> Gate
- C20 pad 2: Gate -> T-
- R3 pad 1: T- -> Gate
- R3 pad 2: Gate -> T-
Routing:
- net Earth: track 295.6 -> 0.00 mm, vias 142 -> 0
- net GND_{24}: track 210.2 -> 0.00 mm, vias 1 -> 0
- net /Soft_Start-24V/AC_{1}: track 178.7 -> 0.00 mm, vias 1 -> 0
- net T-: track 131.1 -> 0.00 mm
- net Earth_Protective: track 117.8 -> 0.00 mm
- net /Soft_Start-24V/~{AC{1}}: track 115.6 -> 0.00 mm
- net ~{PWM1}: track 101.9 -> 0.00 mm
- net 310V: track 97.4 -> 0.00 mm
- net T+: track 88.7 -> 0.00 mm
- net ~{PWM}: track 72.3 -> 0.00 mm
- net Out1: track 71.9 -> 0.00 mm
- net Out+: track 71.8 -> 0.00 mm
- net Out2: track 71.7 -> 0.00 mm
- net Net-(D6-K): track 71.0 -> 0.00 mm
- net Net-(CY1-Pad1): track 63.1 -> 0.00 mm
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- removed copper zone on F.Cu, net 310V
- removed copper zone on B.Cu, net Earth
- removed copper zone on F.Cu, net Earth
- removed copper zone on B.Cu, net GND
- removed copper zone on F.Cu, net GND
- removed copper zone on F.Cu, net Out+
- removed copper zone on B.Cu, net Out-
- removed copper zone on F.Cu, net Out-
- removed copper zone on B.Cu, net Out1
- removed copper zone on F.Cu, net Out1
- removed copper zone on B.Cu, net Out2
- removed copper zone on F.Cu, net Out2
- removed copper zone on F.Cu, net T+
- removed copper zone on B.Cu, net T-

Commit message: Exploração da Placa de Potência
Explorando diferentes posições para os componentes da placa de potência
Parts:
- added D3: US1M, Diode_SMD:D_SMA, F.Cu at (267.1, 40.6)
- added D5: US1M, Diode_SMD:D_SMA, F.Cu at (266.5, 49.3)
- D2: value K7 -> US1M; footprint Diode_SMD:D_SMA_Handsoldering -> Diode_SMD:D_SMA; moved to F.Cu
- D4: value SS16 -> US1M; footprint Diode_SMD:D_SMB -> Diode_SMD:D_SMA; moved to F.Cu
- moved C20 164.7 mm to (310.0, 67.5)
- moved D1 164.7 mm to (314.6, 51.9)
- moved D10 164.7 mm to (302.5, 66.6)
- moved D7 164.7 mm to (277.5, 75.1)
- moved HS1 164.7 mm to (301.5, 50.1)
- moved Q1 164.7 mm to (308.6, 72.6)
- moved Q3 164.7 mm to (283.5, 72.6)
- moved R18 164.7 mm to (276.5, 78.1)
- moved R3 164.7 mm to (310.0, 65.1)
- moved R5 164.7 mm to (296.5, 64.1)
- moved R6 164.7 mm to (300.5, 63.6)
- moved C17 164.7 mm to (306.2, 73.0)
- moved C22 164.7 mm to (278.5, 70.1)
- moved R13 164.7 mm to (275.8, 70.1)
- moved R17 164.7 mm to (272.5, 76.1)
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- renumbered D5 to D10, D10 to D11, D11 to D12, D12 to D13, D13 to D14, D14 to D15, D15 to D16, D16 to D17, D17 to D18, D9 to D6, D3 to D9
Connections:
- C13 pad 1: Net-(D2-K) -> Net-(D5-K)
- C7 pad 1: Net-(D6-K) -> Net-(D3-K)
- D2 pad 1: Net-(D2-K) -> 7V
- D4 pad 1: 7V -> 24V
- D6 pad 1: Net-(D9-K) (its old number) -> Net-(D6-K)
- D6 pad 2: Net-(D9-A) -> Net-(D6-A)
- F2 pad 1: Net-(D6-K) -> Net-(D3-K)
- R12 pad 2: Net-(D2-K) -> Net-(D5-K)
- R15 pad 1: Net-(D6-K) -> Net-(D3-K)
- R7 pad 1: Net-(D6-K) -> Net-(D3-K)
- R7 pad 2: Net-(D9-K) (its old number) -> Net-(D6-K)
- R8 pad 1: Net-(D9-A) -> Net-(D6-A)
- T3 pad 2: Net-(D2-A) -> Net-(T3-Pad2)
- T3 pad 5: Net-(D18-A) -> Net-(D4-A)
- T3 pad 6: Net-(D4-A) -> Net-(D2-A)
- T3 pad 8: Net-(D6-A) -> Net-(D3-A)
- U1 pad 5: Net-(D2-A) -> Net-(T3-Pad2)
- U1 pad 6: Net-(D2-A) -> Net-(T3-Pad2)
- U1 pad 7: Net-(D2-A) -> Net-(T3-Pad2)
- U1 pad 8: Net-(D2-A) -> Net-(T3-Pad2)
- U2 pad 1: Net-(D9-A) -> Net-(D6-A)

Commit message: Adicionada Fuaração
Adicionada furação de montagem na placa de display, 4 furos M3 nos cantos da placa
Parts:
- removed the C14 at (176.1, 43.5)
- removed the D6 at (214.1, 46.9)
- added C14: 47u, Capacitor_THT:CP_Radial_D6.3mm_P2.50mm, F.Cu at (148.3, 65.2)
- added C14: 47u, Capacitor_THT:CP_Radial_D8.0mm_P3.50mm, F.Cu at (145.7, 21.6)
- added C25: 100n, Capacitor_SMD:C_1206_3216Metric_Pad1.33x1.80mm_HandSolder, F.Cu at (156.5, 62.9)
- added D23: US1M, Diode_SMD:D_SMA, F.Cu at (146.6, 28.6)
- added D23: M7, Diode_SMD:D_SMA, F.Cu at (149.6, 59.0)
- added J5: 24V - Trigger, Connector_PinHeader_2.54mm:PinHeader_1x02_P2.54mm_Vertical, B.Cu at (159.0, 38.5)
- C8, C9, D6, R14, R15, R7, R8, U2: moved to F.Cu
- J4: value 24V -> 24V-Cooler
- moved D22 121.9 mm to (131.4, 47.3), turned to 180 degrees
- moved R14 8.10 mm to (225.6, 51.3)
- moved C10 6.57 mm to (148.1, 49.8), turned to 90 degrees
- moved D6 6.50 mm to (207.2, 66.9)
- moved R7 6.50 mm to (213.2, 66.9)
- moved C23 5.74 mm to (160.0, 41.0)
- moved J4 3.01 mm to (158.5, 33.0), turned to 0 degrees
- moved C7 2.22 mm to (213.3, 44.3)
- moved R15 2.21 mm to (218.8, 42.8)
- moved J2 0.62 mm to (247.5, 130.5)
- moved C19 0.58 mm to (260.5, 143.0)
- moved Cx2 0.57 mm to (107.5, 36.5)
- moved C17 0.53 mm to (306.0, 72.5)
- moved C18 0.53 mm to (314.5, 137.0)
- moved C3 0.52 mm to (214.0, 84.0)
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Connections:
- C10 pad 1: 310V -> 310V - APS
- C13 pad 2: 310V -> 310V - APS
- D22 pad 1: unconnected-(D22-+-Pad1) -> 310V - APS
- D22 pad 2: unconnected-(D22---Pad2) -> Earth
- D22 pad 3: unconnected-(D22-Pad3) -> Net-(CY1-Pad1)
- D22 pad 4: unconnected-(D22-Pad4) -> Net-(CY2-Pad2)
- D5 pad 2: 310V -> 310V - APS
- J4 pad 1: 24V -> 24V-Cooler
- R12 pad 1: 310V -> 310V - APS
- T3 pad 1: 310V -> 310V - APS

Commit message: Finalização da Nova Placa de Potência
Dissipadores reorientados e reposicionados para melhor fluxo de ar

Ajuste dos footprints para dissipadores

Adição de resistores na placa de display para melhor proteção do STM32 e redução do brilho da LCD
Parts:
- removed the C14 at (148.3, 65.2)
- removed the C14 at (145.7, 21.6)
- removed the D18 at (177.5, 60.5)
- removed D2: US1M, Diode_SMD:D_SMA
- removed the D22 at (131.4, 47.3)
- removed the D23 at (146.6, 28.6)
- removed the D23 at (149.6, 59.0)
- removed J5: 24V - Trigger, Connector_PinHeader_2.54mm:PinHeader_1x02_P2.54mm_Vertical
- removed U3: ~, Custom_Transformer:EEL25V 6T+6T
- added C14: 47u, Capacitor_THT:CP_Radial_D6.3mm_P2.50mm, F.Cu at (246.6, 42.3)
- added D20: M7, Diode_SMD:D_SMA, B.Cu at (131.8, 50.6)
- added D21: M7, Diode_SMD:D_SMA, B.Cu at (131.7, 57.9)
- added D25: M7, Diode_SMD:D_SMA, F.Cu at (249.5, 54.0)
- added D6: US1M, Diode_SMD:D_SMA, B.Cu at (210.3, 55.8)
- C8, C9, D3, D5, R14, R15, R24, R25, R26, R27, R28, R29, R30, R31, R7, R8, U2: moved to B.Cu
- D7: renamed from D6; moved to B.Cu
- F2: footprint Connector_JST:JST_XH_B2B-XH-A_1x02_P2.50mm_Vertical -> Connector_PinHeader_2.54mm:PinHeader_1x02_P2.54mm_Vertical
- J4: value 24V-Cooler -> 24V; footprint Connector_JST:JST_XH_B2B-XH-A_1x02_P2.50mm_Vertical -> Connector_PinHeader_2.54mm:PinHeader_1x02_P2.54mm_Vertical
- moved D1 190.6 mm to (124.4, 65.5), turned to 90 degrees
- moved C2 170.8 mm to (56.9, 191.3)
- moved C1 170.0 mm to (53.7, 123.8)
- moved D14 168.2 mm to (219.3, 169.1), turned to 0 degrees
- moved C17 160.3 mm to (146.5, 88.6), turned to -90 degrees
- moved C16 156.3 mm to (130.8, 148.2)
- moved C21 156.3 mm to (148.2, 154.2)
- moved D11 156.3 mm to (136.8, 160.7)
- moved Q2 156.3 mm to (107.8, 160.2)
- moved R16 156.3 mm to (148.2, 151.2)
- moved R19 156.3 mm to (132.2, 163.7)
- moved Q4 156.3 mm to (142.8, 160.5)
- moved D9 156.3 mm to (100.3, 159.6)
- moved R1 156.3 mm to (94.3, 161.1)
- moved R2 156.3 mm to (98.8, 163.1)
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- renumbered D7 to D10, D8 to D11, D11 to D12, D12 to D13, D13 to D14, D14 to D15, D15 to D16, D16 to D17, D17 to D18, D18 to D19, D19 to D22, D20 to D23, D21 to D24, D10 to D8
Connections:
- C10 pad 1: 310V - APS -> 310_{Aux}
- C13 pad 1: Net-(D5-K) -> Net-(D3-K)
- C13 pad 2: 310V - APS -> 310_{Aux}
- C7 pad 1: Net-(D3-K) -> Net-(D5-K)
- D5 pad 2: 310V - APS -> Net-(D5-A)
- F2 pad 1: Net-(D3-K) -> Net-(D5-K)
- J4 pad 1: 24V-Cooler -> 24V
- R12 pad 1: 310V - APS -> 310_{Aux}
- R12 pad 2: Net-(D5-K) -> Net-(D3-K)
- R15 pad 1: Net-(D3-K) -> Net-(D5-K)
- R7 pad 1: Net-(D3-K) -> Net-(D5-K)
- T3 pad 1: 310V - APS -> 310_{Aux}
- T3 pad 2: Net-(T3-Pad2) -> Net-(D3-A)
- T3 pad 8: Net-(D3-A) -> Net-(D5-A)
- U1 pad 5: Net-(T3-Pad2) -> Net-(D3-A)
- U1 pad 6: Net-(T3-Pad2) -> Net-(D3-A)
- U1 pad 7: Net-(T3-Pad2) -> Net-(D3-A)
- U1 pad 8: Net-(T3-Pad2) -> Net-(D3-A)
Routing:
- net GND_{24}: track 0.00 -> 175.2 mm
- net 24V: track 0.00 -> 147.8 mm
- net Earth: track 0.00 -> 144.6 mm, vias 0 -> 142
- net Earth_Protective: track 0.00 -> 130.3 mm, vias 0 -> 1
- net /Soft_Start-24V/~{AC{1}}: track 0.00 -> 103.1 mm
- net Out2: track 0.00 -> 82.9 mm
- net /Soft_Start-24V/AC_{1}: track 0.00 -> 75.8 mm, vias 0 -> 1
- net Out1: track 0.00 -> 71.9 mm
- net Out+: track 0.00 -> 71.8 mm
- net Net-(D5-K): track 0.00 -> 70.0 mm
- net Net-(D20-A): track 0.00 -> 68.5 mm
- net GND: track 0.00 -> 66.0 mm, vias 0 -> 9
- net Net-(D21-A): track 0.00 -> 64.0 mm
- net /Soft_Start-24V/AC_{2}: track 0.00 -> 56.8 mm, vias 0 -> 1
- net 310_{Aux}: track 0.00 -> 48.4 mm
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- added copper zone on F.Cu, net 310V
- added copper zone on B.Cu, net Earth
- added copper zone on F.Cu, net Earth
- added copper zone on B.Cu, net GND
- added copper zone on F.Cu, net GND
- added copper zone on F.Cu, net Out+
- added copper zone on B.Cu, net Out-
- added copper zone on F.Cu, net Out-
- added copper zone on B.Cu, net Out1
- added copper zone on F.Cu, net Out1
- added copper zone on B.Cu, net Out2
- added copper zone on F.Cu, net Out2
- added copper zone on F.Cu, net T+
- added copper zone on B.Cu, net T-
Other:
- board size 202.6 x 144.5 mm -> 200 x 180 mm
