File: Kicad - Projects/Inv_Spot_Pot/Inv_Spot_Pot.kicad_pcb (KiCad board)
At the start: 2 copper layers, 202.6 x 144.5 mm, 91 parts, among them J2 PWM, J3 Display_Power, J4 24V, K1 Y14x-1C-xxDS, Q1 40T120, Q2 40T120, Q3 40T120, Q4 40T120, T1 Transformer_1P_2S, U2 LTV-817S

Commit message: Atualizado Modelo 3D
Atualizado Modelo 3D da placa de display, ainda um pouco fora, mas melhorou a visualização da placa.

Listas BOM sendo utilizadas para montar planilha de cotação da placa.
Routing:
- net GND: track 59.8 -> 66.3 mm
Changed lines of the file:
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@@
 		(sheetname "/Power_Supply/")
 		(sheetfile "Sheets/PS-5_15.kicad_sch")
-		(units
-			(unit
-				(name "A")
-				(pins "1" "2" "4" "5" "6" "7" "9" "8")
-			)
-		)
 		(attr through_hole)
 		(duplicate_pad_numbers_are_jumpers no)
 		(fp_line
 			(start 25.62 4.12)
-			(end -5.62 4.12)
+			(end -4.5 4.12)
 			(stroke
 				(width 0.12)
@@
 		(fp_line
 			(start -5.62 -24.12)
-			(end -5.62 4.12)
+			(end 25.62 -24.12)
 			(stroke
 				(width 0.12)
@@
 		)
 		(fp_line
-			(start -5.62 -24.12)
-			(end 25.62 -24.12)
+			(start -4.5 -28.87)
+			(end -4.5 -0.63)
 			(stroke
 				(width 0.12)
@@
 		(fp_line
 			(start 25.75 4.25)
-			(end -5.75 4.25)
+			(end -4.5 4.25)
 			(stroke
 				(width 0.05)
@@
 		(fp_line
 			(start -5.75 -24.25)
-			(end -5.75 4.25)
+			(end 25.75 -24.25)
 			(stroke
 				(width 0.05)
@@
 		)
 		(fp_line
-			(start -5.75 -24.25)
-			(end 25.75 -24.25)
+			(start -4.5 -24.25)
+			(end -4.5 4.25)
 			(stroke
 				(width 0.05)
@@
 		)
 		(fp_line
-			(start -5.5 4)
-			(end -5.5 -24)
+			(start -4.5 4)
+			(end -4.5 -24)
 			(stroke
 				(width 0.1)
@@
 		(fp_line
 			(start 25.5 4)
-			(end -5.5 4)
+			(end -4.5 4)
 			(stroke
 				(width 0.1)
@@
 			)
 		)
+		(dimension
+			(type orthogonal)
+			(layer "User.4")
+			(pts
+				(xy 178.9925 31.17) (xy 178.9925 60.17)
+			)
+			(height 28.25)
+			(orientation 1)
+			(format
+				(prefix "")
+				(suffix "")
+				(units 3)
+				(units_format 0)
+				(precision 4)
+				(suppress_zeroes yes)
+			)
+			(style
+				(thickness 0.1)
+				(arrow_length 1.27)
+				(text_position_mode 0)
+				(arrow_direction outward)
+				(extension_height 0.58642)
+				(extension_offset 0.5)
+				(keep_text_aligned yes)
+			)
+			(gr_text "29"
+				(at 206.0925 45.67 90)
+				(layer "User.4")
+				(effects
+					(font
+						(size 1 1)
+						(thickness 0.15)
+					)
+				)
+			)
+		)
+		(dimension
+			(type orthogonal)
+			(layer "User.4")
+			(pts
+				(xy 197.7425 50.67) (xy 180.2425 50.67)
+			)
+			(height 13.25)
+			(orientation 0)
+			(format
+				(prefix "")
+				(suffix "")
+				(units 3)
+				(units_format 0)
+				(precision 4)
+				(suppress_zeroes yes)
+			)
+			(style
+				(thickness 0.1)
+				(arrow_length 1.27)
+				(text_position_mode 0)
+				(arrow_direction outward)
+				(extension_height 0.58642)
+				(extension_offset 0.5)
+				(keep_text_aligned yes)
+			)
+			(gr_text "17.5"
+				(at 188.9925 62.77 0)
+				(layer "User.4")
+				(effects
+					(font
+						(size 1 1)
+						(thickness 0.15)
+					)
+				)
+			)
+		)
+		(dimension
+			(type orthogonal)
+			(layer "User.4")
+			(pts
+				(xy 197.7425 35.67) (xy 197.7425 40.67)
+			)
+			(height -17.5)
+			(orientation 1)
+			(format
+				(prefix "")
+				(suffix "")
+				(units 3)
+				(units_format 0)
+				(precision 4)
+				(suppress_zeroes yes)
+			)
+			(style
+				(thickness 0.1)
+				(arrow_length 1.27)
+				(text_position_mode 0)
+				(arrow_direction outward)
+				(extension_height 0.58642)
+				(extension_offset 0.5)
+				(keep_text_aligned yes)
+			)
+			(gr_text "5"
+				(at 179.0925 38.17 90)
+				(layer "User.4")
+				(effects
+					(font
+						(size 1 1)
+						(thickness 0.15)
+					)
+				)
+			)
+		)
 		(pad "1" thru_hole rect
 			(at 0 0 270)
@@
 	)
 	(segment
+		(start 197.7725 68.11)
+		(end 197.7425 68.14)
+		(width 1.5)
+		(layer "B.Cu")
+		(net "GND")
+	)
+	(segment
 		(start 215.645151 48.42)
 		(end 215.7425 48.322651)
@@
 	)
 	(segment
+		(start 197.7425 50.67)
+		(end 209.25 50.67)
+		(width 1.5)
+		(layer "B.Cu")
+		(net "GND")
+	)
+	(segment
 		(start 210.2425 37.67)
 		(end 212.7925 37.67)
@@
 	)
 	(segment
-		(start 197.8925 63.09)
-		(end 197.7725 63.21)
+		(start 197.7725 63.21)
+		(end 197.7725 68.11)
 		(width 1.5)
 		(layer "B.Cu")
@@
 	)
 	(segment
-		(start 197.7425 50.67)
-		(end 207.7425 50.67)
+		(start 197.8925 63.09)
+		(end 197.7725 63.21)
 		(width 1.5)
 		(layer "B.Cu")

Commit message: Cotações
Cotações
Parts:
- added CY4: C, Capacitor_THT:C_Disc_D7.0mm_W2.5mm_P5.00mm, F.Cu at (222.7, 78.0)
- added CY5: C, Capacitor_THT:C_Disc_D7.0mm_W2.5mm_P5.00mm, F.Cu at (231.0, 161.0)
- added D22: DF06S, Diode_SMD:Diode_Bridge_OnSemi_SDIP-4L, F.Cu at (242.9, 163.5)
- added R24: 47, Resistor_SMD:R_2512_6332Metric, B.Cu at (156.5, 94.9)
- added R25: 47, Resistor_SMD:R_2512_6332Metric, B.Cu at (156.5, 98.4)
- added R26: 47, Resistor_SMD:R_2512_6332Metric, B.Cu at (181.9, 89.2)
- added R27: 47, Resistor_SMD:R_2512_6332Metric, B.Cu at (181.9, 93.4)
- added R28: 47, Resistor_SMD:R_2512_6332Metric, B.Cu at (190.4, 159.6)
- added R29: 47, Resistor_SMD:R_2512_6332Metric, B.Cu at (190.4, 163.8)
- added R30: 47, Resistor_SMD:R_2512_6332Metric, B.Cu at (150.8, 151.2)
- added R31: 47, Resistor_SMD:R_2512_6332Metric, B.Cu at (150.8, 155.4)
- added U3: ~, Custom_Transformer:EEL25V 6T+6T, F.Cu at (19.6, 102.4)
- C1, C2, C3, C4: value 220u -> 680u
- C13: value 47p -> 4.7n
- C14: moved to F.Cu
- C15, C16, C17, C18: value 100n -> 4.7n; footprint Capacitor_THT:C_Rect_L11.0mm_W5.3mm_P10.00mm_MKT -> Capacitor_THT:C_Disc_D7.0mm_W2.5mm_P5.00mm
- C19, C20, C21, C22: value 100n -> 10n
- D21: footprint LED_THT:LED_D1.8mm_W3.3mm_H2.4mm -> LED_THT:LED_D5.0mm_Clear
- D4: footprint Diode_SMD:D_SOD-128 -> Diode_SMD:D_SMB
- J3: footprint Connector_PinHeader_2.54mm:PinHeader_1x03_P2.54mm_Vertical -> Connector_JST:JST_XH_B3B-XH-A_1x03_P2.50mm_Vertical
- Q1, Q2, Q3, Q4: value 40T120 -> 60N60
- moved C14 145.2 mm to (239.9, 172.1)
Connections:
- C15 pad 1: 310V -> Net-(C15-Pad1)
- C16 pad 1: T- -> Net-(C16-Pad1)
- C17 pad 1: 310V -> Net-(C17-Pad1)
- C18 pad 1: T+ -> Net-(C18-Pad1)
- C20 pad 1: T- -> Gate
- C20 pad 2: Gate -> T-
- R3 pad 1: T- -> Gate
- R3 pad 2: Gate -> T-
Routing:
- net Net-(D2-A): track 28.8 -> 26.7 mm
- net Earth: track 295.6 -> 293.5 mm

Commit message: Adicionada Fuaração
Adicionada furação de montagem na placa de display, 4 furos M3 nos cantos da placa
Parts:
- moved U3 15.0 mm to (34.1, 106.3)
- moved D20 2.62 mm to (48.5, 43.2)
- moved D21 1.29 mm to (42.1, 40.5), turned to 0 degrees
Routing:
- net GND_{24}: track 210.2 -> 175.2 mm
- net 24V: track 160.1 -> 147.8 mm
- net Net-(D21-K): track 4.57 -> 0.00 mm
- net Net-(D19-K): track 12.8 -> 14.2 mm
Other:
- board size 202.6 x 144.5 mm -> 200 x 180 mm
Changed lines of the file:
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@@
 			(outputformat 1)
 			(mirror no)
-			(drillshape 1)
+			(drillshape 0)
 			(scaleselection 1)
-			(outputdirectory "")
+			(outputdirectory "Production")
 		)
 	)
@@
 	(footprint "Custom_Transformer:EEL25V 6T+6T"
 		(layer "F.Cu")
-		(at 19.558855 102.402703 -90)
+		(at 34.066577 106.289071 -90)
 		(property "Reference" "U3"
 			(at 0 0.72 270)
@@
 	(footprint "LED_THT:LED_D5.0mm_Clear"
 		(layer "F.Cu")
-		(at 41.9 41.77 90)
+		(at 42.125 40.5)
 		(descr "LED, diameter 5.0mm, 2 pins, clear, http://cdn-reichelt.de/documents/datenblatt/A500/LL-504BC2E-009.pdf, generated by kicad-footprint-generator")
 		(tags "LED")
 		(property "Reference" "D21"
-			(at 1.27 -3.96 90)
+			(at 1.27 -3.96 0)
 			(layer "F.SilkS")
 			(effects
@@
 		)
 		(property "Value" "LED"
-			(at 1.27 3.96 90)
+			(at 1.27 3.96 0)
 			(layer "F.Fab")
 			(effects
@@
 		)
 		(property "Datasheet" ""
-			(at 0 0 90)
+			(at 0 0 0)
 			(layer "F.Fab")
 			(hide yes)
@@
 		)
 		(property "Description" "Light emitting diode"
-			(at 0 0 90)
+			(at 0 0 0)
 			(layer "F.Fab")
 			(hide yes)
@@
 		)
 		(property "KiLib_Generator" "LED/THT"
-			(at 0 0 90)
+			(at 0 0 0)
 			(layer "F.SilkS")
 			(hide yes)
@@
 		)
 		(property "Sim.Pins" "1=K 2=A"
-			(at 0 0 90)
+			(at 0 0 0)
 			(unlocked yes)
 			(layer "F.Fab")
@@
 		)
 		(fp_text user "${REFERENCE}"
-			(at 1.27 0 90)
+			(at 1.27 0 0)
 			(layer "F.Fab")
 			(effects
@@
 		)
 		(point
-			(at 41.9 40.5)
+			(at 43.395 40.5)
 			(size 2)
 			(layer "F.Fab")
 		)
 		(pad "1" thru_hole rect
-			(at 0 0 90)
+			(at 0 0)
 			(size 1.8 1.8)
 			(drill 0.9)
@@
 		)
 		(pad "2" thru_hole circle
-			(at 2.54 0 90)
+			(at 2.54 0)
 			(size 1.8 1.8)
 			(drill 0.9)
@@
 	(footprint "Diode_SMD:D_SMA"
 		(layer "B.Cu")
-		(at 45.9 43.5 90)
+		(at 48.5 43.2 90)
 		(descr "Diode SMA (DO-214AC)")
 		(tags "Diode SMA (DO-214AC)")
@@
 	)
 	(gr_rect
-		(start 33.18 30.025)
-		(end 235.75 174.5)
+		(start 34.5 30.025)
+		(end 234.5 210.025)
 		(stroke
 			(width 0.05)
@@
 	)
 	(segment
-		(start 47.13 34)
-		(end 41.9 39.23)
-		(width 1.5)
-		(layer "B.Cu")
-		(net "24V")
-	)
-	(segment
 		(start 150 34)
 		(end 47.13 34)
@@
 	)
 	(segment
-		(start 41.895 39.225)
-		(end 41.9 39.23)
-		(width 1.5)
-		(layer "B.Cu")
-		(net "24V")
-	)
-	(segment
-		(start 43.63 39.23)
-		(end 45.9 41.5)
-		(width 1.5)
-		(layer "B.Cu")
-		(net "24V")
-	)
-	(segment
-		(start 41.9 39.23)
-		(end 43.63 39.23)
-		(width 1.5)
-		(layer "B.Cu")
-		(net "24V")
-	)
-	(segment
 		(start 176.7425 61.67)
 		(end 180.2425 58.17)
@@
 	)
 	(segment
-		(start 38.5 54.35)
-		(end 38.5 42.05)
-		(width 1.5)
-		(layer "B.Cu")
-		(net "GND_{24}")
-	)
-	(segment
-		(start 35.5 38.5)
-		(end 35.5 40.5)
-		(width 1.5)
-		(layer "B.Cu")
-		(net "GND_{24}")
-	)
-	(segment
-		(start 35.5 40.5)
-		(end 37.05 42.05)
-		(width 1.5)
-		(layer "B.Cu")
-		(net "GND_{24}")
-	)
-	(segment
 		(start 152.54 34)
 		(end 152.54 32.44)
@@
 	)
 	(segment
-		(start 42.05 31.95)
-		(end 35.5 38.5)
-		(width 1.5)
-		(layer "B.Cu")
-		(net "GND_{24}")
-	)
-	(segment
 		(start 152.54 32.44)
 		(end 152.05 31.95)
@@
 	)
 	(segment
-		(start 44 59.85)
-		(end 38.5 54.35)
-		(width 1.5)
-		(layer "B.Cu")
-		(net "GND_{24}")
-	)
-	(segment
 		(start 44 56.85)
 		(end 44 59.85)
@@
 	)
 	(segment
-		(start 37.05 42.05)
-		(end 38.5 42.05)
-		(width 1.5)
-		(layer "B.Cu")
-		(net "GND_{24}")
-	)
-	(segment
 		(start 198.2425 55.67)
 		(end 208.0425 55.67)
@@
 	)
 	(segment
-		(start 41.32 41.77)
-		(end 38.5 38.95)
-		(width 1.5)
-		(layer "B.Cu")
-		(net "Net-(D21-K)")
-	)
-	(segment
-		(start 41.9 41.77)
-		(end 41.32 41.77)
-		(width 1.5)
-		(layer "B.Cu")
-		(net "Net-(D21-K)")
-	)
-	(segment
 		(start 215.4675 38.995)
 		(end 215.4675 35.17)
@@
 	)
 	(segment
-		(start 45.9 47.75)
+		(start 47.225 52.875)
 		(end 44 49.65)
 		(width 1.5)
@@
 	)
 	(segment
-		(start 45.9 45.5)
-		(end 45.9 47.75)
+		(start 44 49.65)
+		(end 44 52.85)
 		(width 1.5)
 		(layer "B.Cu")
@@
 	)
 	(segment
-		(start 47.225 52.875)
-		(end 44 49.65)
+		(start 45.95 47.75)
+		(end 45.9 47.75)
 		(width 1.5)
 		(layer "B.Cu")
@@
 	)
 	(segment
-		(start 44 49.65)
-		(end 44 52.85)
+		(start 45.9 47.75)
+		(end 44 49.65)
 		(width 1.5)
 		(layer "B.Cu")
@@
 		(width 1.5)
 		(layer "B.Cu")
+		(net "Net-(D19-K)")
+	)
+	(segment
+		(start 48.5 45.2)
+		(end 45.95 47.75)
+		(width 1.5)
+		(layer "B.Cu")

Commit message: Finalização da Nova Placa de Potência
Dissipadores reorientados e reposicionados para melhor fluxo de ar

Ajuste dos footprints para dissipadores

Adição de resistores na placa de display para melhor proteção do STM32 e redução do brilho da LCD
Parts:
- removed Cx2: C, Capacitor_THT:C_Rect_L24.0mm_W8.6mm_P22.50mm_MKT
- removed the D18 at (172.2, 61.7)
- removed D2: K7, Diode_SMD:D_SMA_Handsoldering
- removed the D22 at (242.9, 163.5)
- removed FL1: EMI_Choke, Inductor_THT:Filtro_Choke
- removed U3: ~, Custom_Transformer:EEL25V 6T+6T
- added C25: 100n, Capacitor_SMD:C_1206_3216Metric_Pad1.33x1.80mm_HandSolder, B.Cu at (48.1, 148.8)
- added D20: M7, Diode_SMD:D_SMA, B.Cu at (73.3, 157.0)
- added D21: M7, Diode_SMD:D_SMA, B.Cu at (77.3, 157.1)
- added D25: M7, Diode_SMD:D_SMA, B.Cu at (50.8, 164.1)
- added D3: US1M, Diode_SMD:D_SMA, B.Cu at (56.2, 123.5)
- added D5: US1M, Diode_SMD:D_SMA, B.Cu at (61.5, 90.0)
- added HS4: Heatsink, Custom_Heatsink:Floating_69x33x62mm, F.Cu at (140.5, 87.6)
- added J5: 24V, Connector_PinHeader_2.54mm:PinHeader_1x02_P2.54mm_Vertical, F.Cu at (49.4, 158.5)
- C10: value 47u -> 100u; footprint Capacitor_THT:CP_Radial_D8.0mm_P3.50mm -> Capacitor_THT:CP_Radial_D18.0mm_P7.50mm
- C14: value 100n -> 47u; footprint Capacitor_SMD:C_1206_3216Metric_Pad1.33x1.80mm_HandSolder -> Capacitor_THT:CP_Radial_D6.3mm_P2.50mm
- C19, R4: moved to B.Cu
- D4: value SS16 -> US1M; footprint Diode_SMD:D_SMB -> Diode_SMD:D_SMA; moved to F.Cu
- D6: value SS16 -> US1M; footprint Diode_SMD:D_SOD-128 -> Diode_SMD:D_SMA
- HS1: footprint Heatsink:Heatsink_35x15mm -> Custom_Heatsink:Floating_50x8x62mm
- J3: footprint Connector_JST:JST_XH_B3B-XH-A_1x03_P2.50mm_Vertical -> Connector_PinHeader_2.54mm:PinHeader_1x03_P2.54mm_Vertical
- R24, R25, R26, R27, R28, R29, R30, R31: moved to F.Cu
- moved R9 194.9 mm to (68.8, 233.0), turned to 0 degrees
- moved C14 191.4 mm to (49.4, 153.1), turned to 180 degrees
- moved D24 190.3 mm to (59.5, 230.0), turned to 90 degrees
- moved D23 180.2 mm to (65.2, 222.6), turned to 180 degrees
- moved K1 179.3 mm to (74.0, 231.1), turned to 90 degrees
- moved D22 176.3 mm to (74.1, 228.6), turned to 0 degrees
- moved C8 175.2 mm to (54.4, 64.2), turned to 90 degrees
- moved J3 174.6 mm to (50.9, 69.2), turned to 180 degrees
- moved C24 172.9 mm to (73.9, 225.3), turned to 180 degrees
- moved J4 172.5 mm to (48.9, 173.8), turned to 180 degrees
- moved C9 170.6 mm to (54.4, 69.2), turned to 90 degrees
- moved F2 169.5 mm to (50.9, 76.0), turned to 180 degrees
- moved C23 167.2 mm to (52.3, 172.5), turned to -90 degrees
- moved TH1 166.5 mm to (89.6, 229.6), turned to 90 degrees
- moved R15 164.1 mm to (55.3, 84.1), turned to 180 degrees
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- renumbered D7 to D10, D8 to D11, D10 to D12, D11 to D13, D12 to D14, D13 to D15, D14 to D16, D15 to D17, D16 to D18, D17 to D19, D19 to D22, D20 to D23, D21 to D24, D9 to D7, D5 to D8, D3 to D9
Connections:
- C10 pad 1: 310V -> 310_{Aux}
- C13 pad 2: 310V -> 310_{Aux}
- C14 pad 1: Earth -> 24V-Cooler
- C14 pad 2: Net-(D2-A) -> GND_{24}
- C7 pad 1: Net-(D6-K) -> Net-(D5-K)
- CY1 pad 1: Net-(CY1-Pad1) -> /Soft_Start-24V/AC_{2}
- CY2 pad 2: Net-(CY2-Pad2) -> /Soft_Start-24V/~{AC{1}}
- D1 pad 2: Net-(CY2-Pad2) -> /Soft_Start-24V/AC_{2}
- D1 pad 3: Net-(CY1-Pad1) -> /Soft_Start-24V/~{AC{1}}
- D4 pad 1: 7V -> 24V
- D6 pad 1: Net-(D6-K) -> 7V
- F2 pad 1: Net-(D6-K) -> Net-(D5-K)
- R12 pad 1: 310V -> 310_{Aux}
- R15 pad 1: Net-(D6-K) -> Net-(D5-K)
- R7 pad 1: Net-(D6-K) -> Net-(D5-K)
- T3 pad 1: 310V -> 310_{Aux}
- T3 pad 2: Net-(D2-A) -> Net-(D3-A)
- T3 pad 5: Net-(D18-A) -> Net-(D4-A)
- T3 pad 6: Net-(D4-A) -> Net-(D6-A)
- T3 pad 8: Net-(D6-A) -> Net-(D5-A)
- U1 pad 5: Net-(D2-A) -> Net-(D3-A)
- U1 pad 6: Net-(D2-A) -> Net-(D3-A)
- U1 pad 7: Net-(D2-A) -> Net-(D3-A)
- U1 pad 8: Net-(D2-A) -> Net-(D3-A)
Routing:
- net Out2: track 71.7 -> 271.3 mm
- net Out1: track 71.9 -> 255.6 mm
- net T+: track 88.7 -> 198.3 mm
- net ~{PWM}: track 72.3 -> 166.4 mm
- net T-: track 126.7 -> 219.6 mm, vias 0 -> 2
- net /Soft_Start-24V/AC_{2}: track 56.8 -> 136.3 mm
- net Net-(D6-K): track 71.0 -> 0.00 mm
- net /Soft_Start-24V/~{AC{1}}: track 103.1 -> 171.8 mm
- net Earth: track 293.5 -> 361.4 mm, vias 142 -> 9
- net Net-(CY1-Pad1): track 63.1 -> 0.00 mm
- net 310_{Aux}: track 0.00 -> 61.3 mm
- net Net-(CY2-Pad2): track 58.7 -> 0.00 mm
- net Net-(D5-K): track 0.00 -> 44.7 mm, vias 0 -> 2
- net Earth_Protective: track 130.3 -> 92.1 mm, vias 1 -> 5
- net /PWM_H: track 26.8 -> 0.00 mm, vias 1 -> 0
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- added copper zone on F.Cu, net /Soft_Start-24V/AC_{2}
- added copper zone on F.Cu, net T-
- removed copper zone on B.Cu, net Out-
- removed copper zone on F.Cu, net Out-
- removed copper zone on B.Cu, net T-
Other:
- board size 200 x 180 mm -> 179.5 x 190 mm
