File: Kicad - Projects/Inv_Spot_Pot/Sheets/Soft_Start.kicad_sch (KiCad schematic)
At the start: 4 parts, among them K1 Y14x-1C-xxDS

Commit message: Semi-final Touches
Menu now uses power instead of current

Removed pulsed timing from "CARVAO" and "ARRUELA" operation modes

Added parafix mode

Fixed schematic for output transformer

Added rectification on the output

Trying different power trace geometry in antecipation of voltage spikes
Parts:
- renumbered D16 to D18, D17 to D19
Changed lines of the file:
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@@
 		(in_pos_files yes)
 		(dnp no)
-		(property "Reference" "D17"
+		(property "Reference" "D19"
 			(at 130.556 64.516 0)
 			(show_name no)
@@
 			(project "Inv_Spot_Pot"
 				(path "/e27abe51-96c0-4fdf-ba00-b5a281cd0e9c/e145c09c-6e3a-499a-ba55-638447bfd84b"
-					(reference "D17")
+					(reference "D19")
 					(unit 1)
 				)
@@
 		(in_pos_files yes)
 		(dnp no)
-		(property "Reference" "D16"
+		(property "Reference" "D18"
 			(at 132.588 72.644 0)
 			(show_name no)
@@
 			(project "Inv_Spot_Pot"
 				(path "/e27abe51-96c0-4fdf-ba00-b5a281cd0e9c/e145c09c-6e3a-499a-ba55-638447bfd84b"
-					(reference "D16")
+					(reference "D18")
 					(unit 1)
 				)

Commit message: Adicionado Footprint do Transformador
Footprint do transformador adicionada

Linha dos capacitores XY adicionada

Alteração nas linhas de PWM
Parts:
- added C24: 100n, Capacitor_SMD:C_1206_3216Metric_Pad1.33x1.80mm_HandSolder, symbol Device:C
- added D20: 1N4007, Diode_SMD:D_SMA, symbol Diode:1N4007
- added R9: 2k2, Resistor_SMD:R_1206_3216Metric_Pad1.30x1.75mm_HandSolder, symbol Device:R
- renumbered D18 to D19, D19 to D21
Connections:
- net GND: now also C24.1, R9.2
- net Trigger: now also D20.2 (A)
- net at D19.1 (K), K1.4: now also C24.2, D20.1 (K); no longer D21.1 (K)
- new net: D21.1 (K), R9.1
Other:
- moved on the sheet: D21

Commit message: Cotações
Cotações
Parts:
- D21: footprint LED_THT:LED_D1.8mm_W3.3mm_H2.4mm -> LED_THT:LED_D5.0mm_Clear
Changed lines of the file:
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@@
 			)
 		)
-		(property "Footprint" "LED_THT:LED_D1.8mm_W3.3mm_H2.4mm"
+		(property "Footprint" "LED_THT:LED_D5.0mm_Clear"
 			(at 114.3 55.88 0)
 			(hide yes)

Commit message: Finalização da Nova Placa de Potência
Dissipadores reorientados e reposicionados para melhor fluxo de ar

Ajuste dos footprints para dissipadores

Adição de resistores na placa de display para melhor proteção do STM32 e redução do brilho da LCD
Parts:
- renumbered D19 to D22, D20 to D23, D21 to D24
Changed lines of the file:
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@@
 		)
 		(instances
-			(project "Inv_Spot_Pot - A"
+			(project "Inv_Spot_Pot"
 				(path "/e27abe51-96c0-4fdf-ba00-b5a281cd0e9c/e145c09c-6e3a-499a-ba55-638447bfd84b"
 					(reference "C24")
@@
 		(in_pos_files yes)
 		(dnp no)
-		(property "Reference" "D21"
+		(property "Reference" "D24"
 			(at 114.046 50.546 0)
 			(show_name no)
@@
 		)
 		(instances
-			(project "Inv_Spot_Pot - A"
-				(path "/e27abe51-96c0-4fdf-ba00-b5a281cd0e9c/e145c09c-6e3a-499a-ba55-638447bfd84b"
-					(reference "D21")
+			(project "Inv_Spot_Pot"
+				(path "/e27abe51-96c0-4fdf-ba00-b5a281cd0e9c/e145c09c-6e3a-499a-ba55-638447bfd84b"
+					(reference "D24")
 					(unit 1)
 				)
@@
 		(in_pos_files yes)
 		(dnp no)
-		(property "Reference" "D19"
+		(property "Reference" "D22"
 			(at 132.588 72.644 0)
 			(show_name no)
@@
 		)
 		(instances
-			(project "Inv_Spot_Pot - A"
-				(path "/e27abe51-96c0-4fdf-ba00-b5a281cd0e9c/e145c09c-6e3a-499a-ba55-638447bfd84b"
-					(reference "D19")
+			(project "Inv_Spot_Pot"
+				(path "/e27abe51-96c0-4fdf-ba00-b5a281cd0e9c/e145c09c-6e3a-499a-ba55-638447bfd84b"
+					(reference "D22")
 					(unit 1)
 				)
@@
 		)
 		(instances
-			(project "Inv_Spot_Pot - A"
+			(project "Inv_Spot_Pot"
 				(path "/e27abe51-96c0-4fdf-ba00-b5a281cd0e9c/e145c09c-6e3a-499a-ba55-638447bfd84b"
 					(reference "R9")
@@
 		(in_pos_files yes)
 		(dnp no)
-		(property "Reference" "D20"
+		(property "Reference" "D23"
 			(at 123.698 61.214 0)
 			(show_name no)
@@
 		)
 		(instances
-			(project "Inv_Spot_Pot - A"
-				(path "/e27abe51-96c0-4fdf-ba00-b5a281cd0e9c/e145c09c-6e3a-499a-ba55-638447bfd84b"
-					(reference "D20")
+			(project "Inv_Spot_Pot"
+				(path "/e27abe51-96c0-4fdf-ba00-b5a281cd0e9c/e145c09c-6e3a-499a-ba55-638447bfd84b"
+					(reference "D23")
 					(unit 1)
 				)
@@
 		)
 		(instances
-			(project "Inv_Spot_Pot - A"
+			(project "Inv_Spot_Pot"
 				(path "/e27abe51-96c0-4fdf-ba00-b5a281cd0e9c/e145c09c-6e3a-499a-ba55-638447bfd84b"
 					(reference "TH1")
@@
 		)
 		(instances
-			(project "Inv_Spot_Pot - A"
+			(project "Inv_Spot_Pot"
 				(path "/e27abe51-96c0-4fdf-ba00-b5a281cd0e9c/e145c09c-6e3a-499a-ba55-638447bfd84b"
 					(reference "K1")

Commit message: Finalização - Placa Protótipo
Versão final da placa protótipo - placa já validada

Alterações:
 - Melhoras no plano terra para retorno de potência
 - Blindagem das trilhas de PWM para os IGBTs inferiores
 - Alargamento das trilhas de saída para a retificação

Falta:
 - Colocar todos os SMDs no lado TOP da placa
 - Ajustar posição dos IGBTs e transformador
Parts:
- D22, D23: value 1N4007 -> M7
Changed lines of the file:
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@@
 			)
 		)
-		(property "Value" "1N4007"
+		(property "Value" "M7"
 			(at 129.5401 72.39 90)
 			(hide yes)
@@
 			)
 		)
-		(property "Value" "1N4007"
+		(property "Value" "M7"
 			(at 120.6501 60.96 90)
 			(hide yes)
